File: archive/moin-kastenwagen-pcb 5col/kastenwagen-1840-pcb.kicad_sch (KiCad schematic)
At the start: 197 parts, among them J2 X1224WRS-04-LPV01, J3 Conn_01x04_Pin, U1 SN74LVC1T45DRL, U2 PRTR5V0U2X, U4 XC6206PxxxMR-Regulator_Linear, U5 STM32F072CBT6

Commit message: PCB und Plate bestellfertig
Parts:
- added C3, C4: 100nF, Capacitor_SMD:C_0402_1005Metric, symbol Device:C_Small
- added LED33, LED34: TF_WS2812_1010, TFL:LED_WS2812B_1010_Xinlight, symbol TFLsymbols:TF_WS2812_1010
- BOOT1: Mfr Part (none) -> TS-1187A-B-A-B
- C11, C12, C13, C14, C15, C16, C17, C18, C19, C20, C21, C22, C23, C24, C25, C26, C27, C28, C29, C30, C31, C32, C33, C34, C35, C36, C37, C38, C39, C40, C41, C42: value 100uF -> 100nF
- MX417.275, MX417.625, MX437.225, MX477.200, MX487.200: footprint PCM_marbastlib-mx:SW_MX_HS_S_CPG151101S11_1u -> TFL:SW_MX_HS_CPG151101S11_1u+3d
- S3: footprint PCM_marbastlib-mx:STAB_MX_P_6.25u -> TFL:STAB_MX_P_6.25u_sizelabel
Connections:
- net 5V is gone; now on net +5V: C11.2, C12.2, C13.2, C14.2, C15.2, C16.2, C17.2, C18.2, C19.2, C20.2, C21.2, C22.2, C23.2, C24.2, C25.2, C26.2, C27.2, C28.2, C29.2, C30.2, C31.2, C32.2, C33.2, C34.2, C35.2, C36.2, C37.2, C38.2, C39.2, C40.2, C41.2, C42.2
- net +5V: now also C3.2, C4.2
- net GND: now also LED33.3 (GND), LED34.3 (GND)
- net at LED32.1 (DO): now also LED33.4 (DI); no longer R2.2
- new net: LED33.1 (DO), LED34.4 (DI)
- new net: C3.1, LED33.2 (VDD)
- new net: C4.1, LED34.2 (VDD)
Other:
- moved on the sheet: R2
