File: moin-kastenwagen-pcb/kastenwagen-1840-pcb.kicad_pcb (KiCad board)
At the start: 2 copper layers, 351.4 x 79.8 mm, 204 parts, among them J2 X1224WRS-04-LPV01, J3 Conn_01x04_Pin, U1 SN74LVC1T45DRL, U2 PRTR5V0U2X, U4 XC6206PxxxMR-Regulator_Linear, U5 STM32F072CBT6

Commit message: PCB und Plate bestellfertig
Parts:
- removed MX181: MX-NoLED, TFL:SW_MX_HS_CPG151101S11_1u+3d
- removed RSW100: Rotary_Encoder_Switch, PCM_marbastlib-various:ROT_Alps_EC11E-Switch
- removed the Ref** at (327.9, 136.8)
- removed the Ref** at (275.5, 116.7)
- removed the Ref** at (282.3, 121.0)
- added ?: , , F.Cu at (335.4, 139.3)
- added D34: BAV70, Package_TO_SOT_SMD:SOT-23, B.Cu at (412.1, 141.0)
- added D36: BAV70, Package_TO_SOT_SMD:SOT-23, B.Cu at (391.5, 89.0)
- added D37: BAV70, Package_TO_SOT_SMD:SOT-23, B.Cu at (391.4, 127.3)
- added D38: BAV70, Package_TO_SOT_SMD:SOT-23, B.Cu at (391.4, 108.1)
- added G***: LOGO, Silkscreen:ClackyVectorCu, B.Cu at (368.8, 97.4)
- added MX14: MX-NoLED, TFL:SW_MX_HS_CPG151101S11_1u+3d, B.Cu at (383.4, 90.5)
- added MX18: MX-NoLED, TFL:SW_MX_HS_CPG151101S11_1.75u+3d, B.Cu at (335.8, 90.5)
- added MX32: MX-NoLED, TFL:SW_MX_HS_CPG151101S11_1u+3d, B.Cu at (383.4, 109.5)
- added MX417.3: MX-NoLED, TFL:SW_MX_HS_CPG151101S11_1u+3d, B.Cu at (211.9, 147.6)
- added MX50: MX-NoLED, TFL:SW_MX_HS_CPG151101S11_1u+3d, B.Cu at (383.4, 128.6)
- added MX60: MX-NoLED, TFL:SW_MX_HS_CPG151101S11_1u+3d, B.Cu at (402.4, 147.6)
- added Ref**: Val**, Silkscreen:Moinboards new logo, F.Cu at (273.9, 105.5)
- added Ref**: Val**, Silkscreen:Kastenwagen Logo - Silkscreen mirrored filled, F.Cu at (344.2, 119.0)
- added S6: MX_stab 5, TFL:MXOnly-5U-NoSwitch, F.Cu at (211.9, 147.6)
- moved D9 19.4 mm to (449.2, 89.2)
- moved MX16 19.1 mm to (421.5, 90.5)
- moved MX17 19.1 mm to (440.5, 90.5)
- moved MX34 19.1 mm to (421.5, 109.5)
- moved MX35 19.1 mm to (440.5, 109.5)
- moved MX36 19.1 mm to (459.6, 109.5)
- moved MX487.1 19.1 mm to (459.6, 138.1)
- moved MX52 19.1 mm to (421.5, 128.6)
- moved MX53 19.1 mm to (440.5, 128.6)
- moved MX54 19.1 mm to (459.6, 128.6)
- moved MX61 19.1 mm to (421.5, 147.6)
- moved MX62 19.1 mm to (440.5, 147.6)
- moved MX63 19.1 mm to (459.6, 147.6)
- moved RSW2 19.1 mm to (459.6, 90.5)
- moved S5 19.1 mm to (459.6, 138.1)
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- renumbered C8 to C10, C9 to C11, C10 to C12, C11 to C13, C12 to C14, C13 to C15, C14 to C16, C15 to C17, C16 to C18, C17 to C19, C43 to C2, C18 to C20, C19 to C21, C20 to C22, C21 to C23, C22 to C24, C23 to C25, C24 to C26, C25 to C27, C26 to C28, C27 to C29, C44 to C3, C28 to C30, C29 to C31, C30 to C32, C31 to C33, C32 to C34, C33 to C35, C34 to C36, C35 to C37, C36 to C38, C37 to C39, C45 to C4, C38 to C40, C39 to C41, C40 to C42, C41 to C43, C42 to C44, C3 to C45, C4 to C46, C46 to C5, C47 to C6, C48 to C7, C49 to C8, C2 to C9, D100 to D1, D202 to D10, D203 to D11, D222 to D12, D223 to D13, D242 to D14, D243 to D15, D262 to D16, D272 to D17, D273 to D18, D304 to D19, D101 to D2, D305 to D20, D324 to D21, D325 to D22, D344 to D23, D345 to D24, D364 to D25, D374 to D26, D375 to D27, D406 to D28, D407 to D29, D120 to D3, D437 to D30, D446 to D31, D457 to D32, D1 to D33, D477 to D35, D121 to D4, D140 to D5, D141 to D6, D160 to D7, D170 to D8, D171 to D9, J2 to J1, J3 to J2, MX100 to MX1, MX141 to MX10, MX150 to MX11, MX151 to MX12, MX160 to MX13, MX170 to MX15, MX171 to MX16, MX180 to MX17, MX202 to MX19, MX101 to MX2, MX203 to MX20, MX212 to MX21, MX213 to MX22, MX222 to MX23, MX223 to MX24, MX232 to MX25, MX233 to MX26, MX242 to MX27, MX243 to MX28, MX252 to MX29, MX110 to MX3, MX253 to MX30, MX262 to MX31, MX272 to MX33, MX273 to MX34, MX282 to MX35, MX283 to MX36, MX304 to MX37, MX305 to MX38, MX314 to MX39, MX111 to MX4, MX315 to MX40, MX406.125 to MX406.1, MX324 to MX41, MX416.125 to MX416.1, MX417.275 to MX417.1, MX417.625 to MX417.2, MX325 to MX42, MX334 to MX43, MX437.225 to MX437.1, MX335 to MX44, MX446.125 to MX446.1, MX344 to MX45, MX456.125 to MX456.1, MX345 to MX46, MX354 to MX47, MX477.200 to MX477.1, MX355 to MX48, MX487.200 to MX487.1, MX364 to MX49, MX120 to MX5, MX374 to MX51, MX375 to MX52, MX384 to MX53, MX385 to MX54, MX407 to MX55, MX447 to MX56, MX457 to MX57, MX467 to MX58, MX476 to MX59, MX121 to MX6, MX477 to MX61, MX486 to MX62, MX487 to MX63, MX130 to MX7, MX131 to MX8, MX140 to MX9, R8 to R1, R9 to R2, R1 to R3, R2 to R4, RSW181 to RSW2, S4 to S1, S1 to S3, S3 to S4, U5 to U1, U4 to U3, U1 to U4
Connections:
- D33 pad 2: Net-(MX477-ROW) -> unconnected-(D33-A-Pad2)
- LED34 pad 1: unconnected-(LED34-DO-Pad1) -> Net-(LED34-DO)
- MX15 pad 1: Col13 -> Col14
- MX16 pad 1: Col14 -> Col15
- MX17 pad 1: Col15 -> Col16
- MX33 pad 1: Col13 -> Col14
- MX34 pad 1: Col14 -> Col15
- MX35 pad 1: Col15 -> Col16
- MX36 pad 1: Col16 -> Col17
- MX446.1 pad 1: Col8 -> Col7
- MX456.1 pad 1: Col10 -> Col9
- MX477.1 pad 2: Net-(MX477-ROW) -> Net-(MX477.1-ROW)
- MX487.1 pad 1: Col16 -> Col17
- MX51 pad 1: Col13 -> Col14
- MX52 pad 1: Col14 -> Col15
- MX53 pad 1: Col15 -> Col16
- MX54 pad 1: Col16 -> Col17
- MX56 pad 1: Col9 -> Col8
- MX57 pad 1: Col11 -> Col10
- MX58 pad 1: Col12 -> Col11
- MX59 pad 1: Col13 -> Col12
- MX61 pad 1: Col14 -> Col15
- MX61 pad 2: Net-(MX477-ROW) -> Net-(MX61-ROW)
- MX62 pad 1: Col15 -> Col16
- MX63 pad 1: Col16 -> Col17
- R4 pad 2: unconnected-(R2-Pad2) -> Net-(LED34-DO)
- RSW2 pad S2: Col16 -> Col17
- U1 pad 13: unconnected-(U5-PA3-Pad13) -> Col17
- U1 pad 14: Rotary0B -> unconnected-(U1-PA4-Pad14)
- U1 pad 15: Rotary0A -> unconnected-(U1-PA5-Pad15)
Routing:
- net Rotary0B: track 281.7 -> 0.00 mm, vias 1 -> 0
- net Rotary0A: track 277.4 -> 0.00 mm, vias 1 -> 0
- net Col17: track 0.00 -> 199.5 mm, vias 0 -> 2
- net Row1: track 382.1 -> 418.1 mm
- net Row0: track 418.0 -> 445.5 mm
- net Col7: track 144.0 -> 169.9 mm
- net Col13: track 88.8 -> 64.3 mm
- net Net-(MX417.2-ROW): track 29.6 -> 53.9 mm
- net Col16: track 164.1 -> 140.6 mm
- net Net-(MX477-ROW): track 23.2 -> 0.00 mm
- net Col12: track 77.4 -> 98.1 mm
- net Col10: track 104.7 -> 124.9 mm
- net Rotary1A: track 118.0 -> 137.0 mm
- net Rotary1B: track 113.3 -> 132.3 mm
- net Row3: track 399.0 -> 416.5 mm
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Other:
- board size 351.4 x 79.8 mm -> 370.2 x 79.8 mm
- board text added: "1.75 BS"
- board text added: "5u"
- board text added: "Kastenwagen Alu BAN v1.0 by Technofrikus, based on Kastenwagen by NoPunIn10did"
- board text added: "LAE"
- board text removed: "Kastenwagen Alu PCB v1.0 by Technofrikus Based on Kastenwagen by NoPunIn10Did"
