File: moin-kastenwagen-pcb/kastenwagen-1840-pcb.kicad_sch (KiCad schematic)
At the start: 201 parts, among them J2 X1224WRS-04-LPV01, J3 Conn_01x04_Pin, U1 SN74LVC1T45DRL, U2 PRTR5V0U2X, U4 XC6206PxxxMR-Regulator_Linear, U5 STM32F072CBT6

Commit message: Untestested v1 finished. Ready for Protos.
Parts:
- BOOT1: Mfr Part (none) -> TS-1187A-B-A-B
- C11, C12, C13, C14, C15, C16, C17, C18, C19, C20, C21, C22, C23, C24, C25, C26, C27, C28, C29, C3, C30, C31, C32, C33, C34, C35, C36, C37, C38, C39, C4, C40, C41, C42: value 100uF -> 100nF
- MX417.275, MX417.625, MX437.225, MX477.200, MX487.200: footprint PCM_marbastlib-mx:SW_MX_HS_S_CPG151101S11_1u -> TFL:SW_MX_HS_CPG151101S11_1u+3d

Commit message: PCB und Plate bestellfertig
Parts:
- removed MX181: MX-NoLED, TFL:SW_MX_HS_CPG151101S11_1u+3d, symbol MX_Alps_Hybrid:MX-NoLED
- removed RSW100: Rotary_Encoder_Switch, PCM_marbastlib-various:ROT_Alps_EC11E-Switch, symbol nopun-custom-mx-symbols:Rotary_Encoder_Switch-Device
- added D34, D36, D37, D38: BAV70, Package_TO_SOT_SMD:SOT-23, symbol Diode:BAV70
- added MX14, MX32, MX417.3, MX50, MX60: MX-NoLED, TFL:SW_MX_HS_CPG151101S11_1u+3d, symbol MX_Alps_Hybrid:MX-NoLED
- added MX18: MX-NoLED, PCM_marbastlib-mx:SW_MX_1u, symbol MX_Alps_Hybrid:MX-NoLED
- added S6: MX_stab 5, TFL:MXOnly-5U-NoSwitch, symbol PCM_marbastlib-mx:MX_stab
- BOOT1: LCSC (none) -> C318884; MPN (none) -> TS-1187A-B-A-B; Manufacturer (none) -> XKB Connection; Original (none) -> N; Purchase Link (none) -> https://www.lcsc.com/product-detail/C318884.html?s_z=n_C318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
- C1: Manufacturer (none) -> Samsung Electro-Mechanics; Original (none) -> N; Purchase Link (none) -> https://www.lcsc.com/product-detail/C307331.html?s_z=n_C307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
- C10: renamed from C8; MPN (none) -> CL05B104KB54PNC; Manufacturer (none) -> Samsung Electro-Mechanics; Original (none) -> N; Purchase Link (none) -> https://www.lcsc.com/product-detail/C307331.html?s_z=n_C307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
- C11: renamed from C9; LCSC C307331 -> C52923; MPN (none) -> CL05A105KA5NQNC; Manufacturer (none) -> Samsung Electro-Mechanics; Original (none) -> N; Purchase Link (none) -> https://www.lcsc.com/product-detail/C52923.html?s_z=n_C52923
- C12: renamed from C10; LCSC C307331 -> C52923; MPN (none) -> CL05A105KA5NQNC; Manufacturer (none) -> Samsung Electro-Mechanics; Original (none) -> N; Purchase Link (none) -> https://www.lcsc.com/product-detail/C52923.html?s_z=n_C52923
- C13: renamed from C11; LCSC (none) -> C307331; MPN (none) -> CL05B104KB54PNC; Manufacturer (none) -> Samsung Electro-Mechanics; Original (none) -> N; Purchase Link (none) -> https://www.lcsc.com/product-detail/C307331.html?s_z=n_C307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
- C14: renamed from C12; LCSC (none) -> C307331; MPN (none) -> CL05B104KB54PNC; Manufacturer (none) -> Samsung Electro-Mechanics; Original (none) -> N; Purchase Link (none) -> https://www.lcsc.com/product-detail/C307331.html?s_z=n_C307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
- C15: renamed from C13; LCSC (none) -> C307331; MPN (none) -> CL05B104KB54PNC; Manufacturer (none) -> Samsung Electro-Mechanics; Original (none) -> N; Purchase Link (none) -> https://www.lcsc.com/product-detail/C307331.html?s_z=n_C307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
- C16: renamed from C14; LCSC (none) -> C307331; MPN (none) -> CL05B104KB54PNC; Manufacturer (none) -> Samsung Electro-Mechanics; Original (none) -> N; Purchase Link (none) -> https://www.lcsc.com/product-detail/C307331.html?s_z=n_C307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
- C17: renamed from C15; LCSC (none) -> C307331; MPN (none) -> CL05B104KB54PNC; Manufacturer (none) -> Samsung Electro-Mechanics; Original (none) -> N; Purchase Link (none) -> https://www.lcsc.com/product-detail/C307331.html?s_z=n_C307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
- C18: renamed from C16; LCSC (none) -> C307331; MPN (none) -> CL05B104KB54PNC; Manufacturer (none) -> Samsung Electro-Mechanics; Original (none) -> N; Purchase Link (none) -> https://www.lcsc.com/product-detail/C307331.html?s_z=n_C307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
- C19: renamed from C17; LCSC (none) -> C307331; MPN (none) -> CL05B104KB54PNC; Manufacturer (none) -> Samsung Electro-Mechanics; Original (none) -> N; Purchase Link (none) -> https://www.lcsc.com/product-detail/C307331.html?s_z=n_C307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
- C2: renamed from C43; Manufacturer (none) -> Samsung Electro-Mechanics; Original (none) -> N; Purchase Link (none) -> https://www.lcsc.com/product-detail/C307331.html?s_z=n_C307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
- C20: renamed from C18; LCSC (none) -> C307331; MPN (none) -> CL05B104KB54PNC; Manufacturer (none) -> Samsung Electro-Mechanics; Original (none) -> N; Purchase Link (none) -> https://www.lcsc.com/product-detail/C307331.html?s_z=n_C307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
- C21: renamed from C19; LCSC (none) -> C307331; MPN (none) -> CL05B104KB54PNC; Manufacturer (none) -> Samsung Electro-Mechanics; Original (none) -> N; Purchase Link (none) -> https://www.lcsc.com/product-detail/C307331.html?s_z=n_C307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
- C22: renamed from C20; LCSC (none) -> C307331; MPN (none) -> CL05B104KB54PNC; Manufacturer (none) -> Samsung Electro-Mechanics; Original (none) -> N; Purchase Link (none) -> https://www.lcsc.com/product-detail/C307331.html?s_z=n_C307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
- C23: renamed from C21; LCSC (none) -> C307331; MPN (none) -> CL05B104KB54PNC; Manufacturer (none) -> Samsung Electro-Mechanics; Original (none) -> N; Purchase Link (none) -> https://www.lcsc.com/product-detail/C307331.html?s_z=n_C307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
- C24: renamed from C22; LCSC (none) -> C307331; MPN (none) -> CL05B104KB54PNC; Manufacturer (none) -> Samsung Electro-Mechanics; Original (none) -> N; Purchase Link (none) -> https://www.lcsc.com/product-detail/C307331.html?s_z=n_C307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
- C25: renamed from C23; LCSC (none) -> C307331; MPN (none) -> CL05B104KB54PNC; Manufacturer (none) -> Samsung Electro-Mechanics; Original (none) -> N; Purchase Link (none) -> https://www.lcsc.com/product-detail/C307331.html?s_z=n_C307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
- C26: renamed from C24; LCSC (none) -> C307331; MPN (none) -> CL05B104KB54PNC; Manufacturer (none) -> Samsung Electro-Mechanics; Original (none) -> N; Purchase Link (none) -> https://www.lcsc.com/product-detail/C307331.html?s_z=n_C307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
- C27: renamed from C25; LCSC (none) -> C307331; MPN (none) -> CL05B104KB54PNC; Manufacturer (none) -> Samsung Electro-Mechanics; Original (none) -> N; Purchase Link (none) -> https://www.lcsc.com/product-detail/C307331.html?s_z=n_C307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
- C28: renamed from C26; LCSC (none) -> C307331; MPN (none) -> CL05B104KB54PNC; Manufacturer (none) -> Samsung Electro-Mechanics; Original (none) -> N; Purchase Link (none) -> https://www.lcsc.com/product-detail/C307331.html?s_z=n_C307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
- C29: renamed from C27; LCSC (none) -> C307331; MPN (none) -> CL05B104KB54PNC; Manufacturer (none) -> Samsung Electro-Mechanics; Original (none) -> N; Purchase Link (none) -> https://www.lcsc.com/product-detail/C307331.html?s_z=n_C307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
- C3: renamed from C44; Manufacturer (none) -> Samsung Electro-Mechanics; Original (none) -> N; Purchase Link (none) -> https://www.lcsc.com/product-detail/C23733.html?s_z=n_C23733
- C30: renamed from C28; LCSC (none) -> C307331; MPN (none) -> CL05B104KB54PNC; Manufacturer (none) -> Samsung Electro-Mechanics; Original (none) -> N; Purchase Link (none) -> https://www.lcsc.com/product-detail/C307331.html?s_z=n_C307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
- C31: renamed from C29; LCSC (none) -> C307331; MPN (none) -> CL05B104KB54PNC; Manufacturer (none) -> Samsung Electro-Mechanics; Original (none) -> N; Purchase Link (none) -> https://www.lcsc.com/product-detail/C307331.html?s_z=n_C307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
- C32: renamed from C30; LCSC (none) -> C307331; MPN (none) -> CL05B104KB54PNC; Manufacturer (none) -> Samsung Electro-Mechanics; Original (none) -> N; Purchase Link (none) -> https://www.lcsc.com/product-detail/C307331.html?s_z=n_C307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
- C33: renamed from C31; LCSC (none) -> C307331; MPN (none) -> CL05B104KB54PNC; Manufacturer (none) -> Samsung Electro-Mechanics; Original (none) -> N; Purchase Link (none) -> https://www.lcsc.com/product-detail/C307331.html?s_z=n_C307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
- C34: renamed from C32; LCSC (none) -> C307331; MPN (none) -> CL05B104KB54PNC; Manufacturer (none) -> Samsung Electro-Mechanics; Original (none) -> N; Purchase Link (none) -> https://www.lcsc.com/product-detail/C307331.html?s_z=n_C307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
- C35: renamed from C33; LCSC (none) -> C307331; MPN (none) -> CL05B104KB54PNC; Manufacturer (none) -> Samsung Electro-Mechanics; Original (none) -> N; Purchase Link (none) -> https://www.lcsc.com/product-detail/C307331.html?s_z=n_C307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
- C36: renamed from C34; LCSC (none) -> C307331; MPN (none) -> CL05B104KB54PNC; Manufacturer (none) -> Samsung Electro-Mechanics; Original (none) -> N; Purchase Link (none) -> https://www.lcsc.com/product-detail/C307331.html?s_z=n_C307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
- C37: renamed from C35; LCSC (none) -> C307331; MPN (none) -> CL05B104KB54PNC; Manufacturer (none) -> Samsung Electro-Mechanics; Original (none) -> N; Purchase Link (none) -> https://www.lcsc.com/product-detail/C307331.html?s_z=n_C307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
- C38: renamed from C36; LCSC (none) -> C307331; MPN (none) -> CL05B104KB54PNC; Manufacturer (none) -> Samsung Electro-Mechanics; Original (none) -> N; Purchase Link (none) -> https://www.lcsc.com/product-detail/C307331.html?s_z=n_C307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
- C39: renamed from C37; LCSC (none) -> C307331; MPN (none) -> CL05B104KB54PNC; Manufacturer (none) -> Samsung Electro-Mechanics; Original (none) -> N; Purchase Link (none) -> https://www.lcsc.com/product-detail/C307331.html?s_z=n_C307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
- C4: renamed from C45; Manufacturer (none) -> Samsung Electro-Mechanics; Original (none) -> N; Purchase Link (none) -> https://www.lcsc.com/product-detail/C307331.html?s_z=n_C307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
- C40: renamed from C38; LCSC (none) -> C307331; MPN (none) -> CL05B104KB54PNC; Manufacturer (none) -> Samsung Electro-Mechanics; Original (none) -> N; Purchase Link (none) -> https://www.lcsc.com/product-detail/C307331.html?s_z=n_C307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
- C41: renamed from C39; LCSC (none) -> C307331; MPN (none) -> CL05B104KB54PNC; Manufacturer (none) -> Samsung Electro-Mechanics; Original (none) -> N; Purchase Link (none) -> https://www.lcsc.com/product-detail/C307331.html?s_z=n_C307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
- C42: renamed from C40; LCSC (none) -> C307331; MPN (none) -> CL05B104KB54PNC; Manufacturer (none) -> Samsung Electro-Mechanics; Original (none) -> N; Purchase Link (none) -> https://www.lcsc.com/product-detail/C307331.html?s_z=n_C307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
- C43: renamed from C41; LCSC (none) -> C307331; MPN (none) -> CL05B104KB54PNC; Manufacturer (none) -> Samsung Electro-Mechanics; Original (none) -> N; Purchase Link (none) -> https://www.lcsc.com/product-detail/C307331.html?s_z=n_C307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
- C44: renamed from C42; LCSC (none) -> C307331; MPN (none) -> CL05B104KB54PNC; Manufacturer (none) -> Samsung Electro-Mechanics; Original (none) -> N; Purchase Link (none) -> https://www.lcsc.com/product-detail/C307331.html?s_z=n_C307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
- C45: renamed from C3; LCSC (none) -> C307331; MPN (none) -> CL05B104KB54PNC; Manufacturer (none) -> Samsung Electro-Mechanics; Original (none) -> N; Purchase Link (none) -> https://www.lcsc.com/product-detail/C307331.html?s_z=n_C307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
- C46: renamed from C4; LCSC (none) -> C307331; MPN (none) -> CL05B104KB54PNC; Manufacturer (none) -> Samsung Electro-Mechanics; Original (none) -> N; Purchase Link (none) -> https://www.lcsc.com/product-detail/C307331.html?s_z=n_C307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
- C5: renamed from C46; Manufacturer (none) -> Samsung Electro-Mechanics; Original (none) -> N; Purchase Link (none) -> https://www.lcsc.com/product-detail/C15195.html?s_z=n_C15195
- C6: renamed from C47; Manufacturer (none) -> Samsung Electro-Mechanics; Original (none) -> N; Purchase Link (none) -> https://www.lcsc.com/product-detail/C52923.html?s_z=n_C52923
- C7: renamed from C48; Manufacturer (none) -> Samsung Electro-Mechanics; Original (none) -> N; Purchase Link (none) -> https://www.lcsc.com/product-detail/C307331.html?s_z=n_C307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
- C8: renamed from C49; Manufacturer (none) -> Samsung Electro-Mechanics; Original (none) -> N; Purchase Link (none) -> https://www.lcsc.com/product-detail/C23733.html?s_z=n_C23733
- C9: renamed from C2; Manufacturer (none) -> Samsung Electro-Mechanics; Original (none) -> N; Purchase Link (none) -> https://www.lcsc.com/product-detail/C307331.html?s_z=n_C307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
- D1: renamed from D100; LCSC (none) -> C68978; MPN (none) -> BAV70; Manufacturer (none) -> JSCJ; Original (none) -> N; Purchase Link (none) -> https://www.lcsc.com/product-detail/C68978.html?s_z=n_C68978
- D10: renamed from D202; LCSC (none) -> C68978; MPN (none) -> BAV70; Manufacturer (none) -> JSCJ; Original (none) -> N; Purchase Link (none) -> https://www.lcsc.com/product-detail/C68978.html?s_z=n_C68978
- D11: renamed from D203; LCSC (none) -> C68978; MPN (none) -> BAV70; Manufacturer (none) -> JSCJ; Original (none) -> N; Purchase Link (none) -> https://www.lcsc.com/product-detail/C68978.html?s_z=n_C68978
- D12: renamed from D222; LCSC (none) -> C68978; MPN (none) -> BAV70; Manufacturer (none) -> JSCJ; Original (none) -> N; Purchase Link (none) -> https://www.lcsc.com/product-detail/C68978.html?s_z=n_C68978
- D13: renamed from D223; LCSC (none) -> C68978; MPN (none) -> BAV70; Manufacturer (none) -> JSCJ; Original (none) -> N; Purchase Link (none) -> https://www.lcsc.com/product-detail/C68978.html?s_z=n_C68978
- D14: renamed from D242; LCSC (none) -> C68978; MPN (none) -> BAV70; Manufacturer (none) -> JSCJ; Original (none) -> N; Purchase Link (none) -> https://www.lcsc.com/product-detail/C68978.html?s_z=n_C68978
- D15: renamed from D243; LCSC (none) -> C68978; MPN (none) -> BAV70; Manufacturer (none) -> JSCJ; Original (none) -> N; Purchase Link (none) -> https://www.lcsc.com/product-detail/C68978.html?s_z=n_C68978
- D16: renamed from D262; LCSC (none) -> C68978; MPN (none) -> BAV70; Manufacturer (none) -> JSCJ; Original (none) -> N; Purchase Link (none) -> https://www.lcsc.com/product-detail/C68978.html?s_z=n_C68978
- D17: renamed from D272; LCSC (none) -> C68978; MPN (none) -> BAV70; Manufacturer (none) -> JSCJ; Original (none) -> N; Purchase Link (none) -> https://www.lcsc.com/product-detail/C68978.html?s_z=n_C68978
- D18: renamed from D273; LCSC (none) -> C68978; MPN (none) -> BAV70; Manufacturer (none) -> JSCJ; Original (none) -> N; Purchase Link (none) -> https://www.lcsc.com/product-detail/C68978.html?s_z=n_C68978
- D19: renamed from D304; LCSC (none) -> C68978; MPN (none) -> BAV70; Manufacturer (none) -> JSCJ; Original (none) -> N; Purchase Link (none) -> https://www.lcsc.com/product-detail/C68978.html?s_z=n_C68978
- D2: renamed from D101; LCSC (none) -> C68978; MPN (none) -> BAV70; Manufacturer (none) -> JSCJ; Original (none) -> N; Purchase Link (none) -> https://www.lcsc.com/product-detail/C68978.html?s_z=n_C68978
- D20: renamed from D305; LCSC (none) -> C68978; MPN (none) -> BAV70; Manufacturer (none) -> JSCJ; Original (none) -> N; Purchase Link (none) -> https://www.lcsc.com/product-detail/C68978.html?s_z=n_C68978
- D21: renamed from D324; LCSC (none) -> C68978; MPN (none) -> BAV70; Manufacturer (none) -> JSCJ; Original (none) -> N; Purchase Link (none) -> https://www.lcsc.com/product-detail/C68978.html?s_z=n_C68978
- D22: renamed from D325; LCSC (none) -> C68978; MPN (none) -> BAV70; Manufacturer (none) -> JSCJ; Original (none) -> N; Purchase Link (none) -> https://www.lcsc.com/product-detail/C68978.html?s_z=n_C68978
- D23: renamed from D344; LCSC (none) -> C68978; MPN (none) -> BAV70; Manufacturer (none) -> JSCJ; Original (none) -> N; Purchase Link (none) -> https://www.lcsc.com/product-detail/C68978.html?s_z=n_C68978
- D24: renamed from D345; LCSC (none) -> C68978; MPN (none) -> BAV70; Manufacturer (none) -> JSCJ; Original (none) -> N; Purchase Link (none) -> https://www.lcsc.com/product-detail/C68978.html?s_z=n_C68978
- D25: renamed from D364; LCSC (none) -> C68978; MPN (none) -> BAV70; Manufacturer (none) -> JSCJ; Original (none) -> N; Purchase Link (none) -> https://www.lcsc.com/product-detail/C68978.html?s_z=n_C68978
- D26: renamed from D374; LCSC (none) -> C68978; MPN (none) -> BAV70; Manufacturer (none) -> JSCJ; Original (none) -> N; Purchase Link (none) -> https://www.lcsc.com/product-detail/C68978.html?s_z=n_C68978
- D27: renamed from D375; LCSC (none) -> C68978; MPN (none) -> BAV70; Manufacturer (none) -> JSCJ; Original (none) -> N; Purchase Link (none) -> https://www.lcsc.com/product-detail/C68978.html?s_z=n_C68978
- D28: renamed from D406; LCSC (none) -> C68978; MPN (none) -> BAV70; Manufacturer (none) -> JSCJ; Original (none) -> N; Purchase Link (none) -> https://www.lcsc.com/product-detail/C68978.html?s_z=n_C68978
- D29: renamed from D407; LCSC (none) -> C68978; MPN (none) -> BAV70; Manufacturer (none) -> JSCJ; Original (none) -> N; Purchase Link (none) -> https://www.lcsc.com/product-detail/C68978.html?s_z=n_C68978
- D3: renamed from D120; LCSC (none) -> C68978; MPN (none) -> BAV70; Manufacturer (none) -> JSCJ; Original (none) -> N; Purchase Link (none) -> https://www.lcsc.com/product-detail/C68978.html?s_z=n_C68978
- D30: renamed from D437; LCSC (none) -> C68978; MPN (none) -> BAV70; Manufacturer (none) -> JSCJ; Original (none) -> N; Purchase Link (none) -> https://www.lcsc.com/product-detail/C68978.html?s_z=n_C68978
- D31: renamed from D446; LCSC (none) -> C68978; MPN (none) -> BAV70; Manufacturer (none) -> JSCJ; Original (none) -> N; Purchase Link (none) -> https://www.lcsc.com/product-detail/C68978.html?s_z=n_C68978
- D32: renamed from D457; LCSC (none) -> C68978; MPN (none) -> BAV70; Manufacturer (none) -> JSCJ; Original (none) -> N; Purchase Link (none) -> https://www.lcsc.com/product-detail/C68978.html?s_z=n_C68978
- D33: renamed from D1; MPN (none) -> BAV70; Manufacturer (none) -> JSCJ; Original (none) -> N; Purchase Link (none) -> https://www.lcsc.com/product-detail/C68978.html?s_z=n_C68978
- D35: renamed from D477; MPN (none) -> BAV70; Manufacturer (none) -> JSCJ; Original (none) -> N; Purchase Link (none) -> https://www.lcsc.com/product-detail/C68978.html?s_z=n_C68978
- D4: renamed from D121; LCSC (none) -> C68978; MPN (none) -> BAV70; Manufacturer (none) -> JSCJ; Original (none) -> N; Purchase Link (none) -> https://www.lcsc.com/product-detail/C68978.html?s_z=n_C68978
- D5: renamed from D140; LCSC (none) -> C68978; MPN (none) -> BAV70; Manufacturer (none) -> JSCJ; Original (none) -> N; Purchase Link (none) -> https://www.lcsc.com/product-detail/C68978.html?s_z=n_C68978
- D6: renamed from D141; LCSC (none) -> C68978; MPN (none) -> BAV70; Manufacturer (none) -> JSCJ; Original (none) -> N; Purchase Link (none) -> https://www.lcsc.com/product-detail/C68978.html?s_z=n_C68978
- D7: renamed from D160; LCSC (none) -> C68978; MPN (none) -> BAV70; Manufacturer (none) -> JSCJ; Original (none) -> N; Purchase Link (none) -> https://www.lcsc.com/product-detail/C68978.html?s_z=n_C68978
- D8: renamed from D170; LCSC (none) -> C68978; MPN (none) -> BAV70; Manufacturer (none) -> JSCJ; Original (none) -> N; Purchase Link (none) -> https://www.lcsc.com/product-detail/C68978.html?s_z=n_C68978
- D9: renamed from D171; LCSC (none) -> C68978; MPN (none) -> BAV70; Manufacturer (none) -> JSCJ; Original (none) -> N; Purchase Link (none) -> https://www.lcsc.com/product-detail/C68978.html?s_z=n_C68978
- F1: MPN (none) -> ASMD1206-150; Manufacturer (none) -> JDTfuse; Original (none) -> N; Purchase Link (none) -> https://www.lcsc.com/product-detail/C135341.html?s_z=n_C135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
- J1: renamed from J2; MPN (none) -> 781710004; Original (none) -> Y; Purchase Link (none) -> https://www.lcsc.com/product-detail/C588524.html?s_z=n_C588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
- J2: renamed from J3; now not fitted
- LED1, LED10, LED11, LED12, LED13, LED14, LED15, LED16, LED17, LED18, LED19, LED2, LED20, LED21, LED22, LED23, LED24, LED25, LED26, LED27, LED28, LED29, LED3, LED30, LED31, LED32, LED33, LED34, LED4, LED5, LED6, LED7, LED8, LED9: LCSC (none) -> C5349953; MPN (none) -> XL-1010RGBC-2812B; Manufacturer (none) -> XINGLIGHT; Original (none) -> Y; Purchase Link (none) -> https://www.lcsc.com/product-detail/C5349953.html?s_z=n_C53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
- MX1: renamed from MX100; now not fitted
- MX10: renamed from MX141; now not fitted
- MX11: renamed from MX150; now not fitted
- MX12: renamed from MX151; now not fitted
- MX13: renamed from MX160; now not fitted
- MX15: renamed from MX170; now not fitted
- MX16: renamed from MX171; now not fitted
- MX17: renamed from MX180; now not fitted
- MX19: renamed from MX202; now not fitted
- MX2: renamed from MX101; now not fitted
- MX20: renamed from MX203; now not fitted
- MX21: renamed from MX212; now not fitted
- MX22: renamed from MX213; now not fitted
- MX23: renamed from MX222; now not fitted
- MX24: renamed from MX223; now not fitted
- MX25: renamed from MX232; now not fitted
- MX26: renamed from MX233; now not fitted
- MX27: renamed from MX242; now not fitted
- MX28: renamed from MX243; now not fitted
- MX29: renamed from MX252; now not fitted
- MX3: renamed from MX110; now not fitted
- MX30: renamed from MX253; now not fitted
- MX31: renamed from MX262; now not fitted
- MX33: renamed from MX272; now not fitted
- MX34: renamed from MX273; now not fitted
- MX35: renamed from MX282; now not fitted
- MX36: renamed from MX283; now not fitted
- MX37: renamed from MX304; now not fitted
- MX38: renamed from MX305; now not fitted
- MX39: renamed from MX314; now not fitted
- MX4: renamed from MX111; now not fitted
- MX40: renamed from MX315; now not fitted
- MX406.1: renamed from MX406.125; now not fitted
- MX41: renamed from MX324; now not fitted
- MX416.1: renamed from MX416.125; now not fitted
- MX417.1: renamed from MX417.275; now not fitted
- MX417.2: renamed from MX417.625; now not fitted
- MX42: renamed from MX325; now not fitted
- MX43: renamed from MX334; now not fitted
- MX437.1: renamed from MX437.225; now not fitted
- MX44: renamed from MX335; now not fitted
- MX446.1: renamed from MX446.125; now not fitted
- MX45: renamed from MX344; now not fitted
- MX456.1: renamed from MX456.125; now not fitted
- MX46: renamed from MX345; now not fitted
- MX47: renamed from MX354; now not fitted
- MX477.1: renamed from MX477.200; now not fitted
- MX48: renamed from MX355; now not fitted
- MX487.1: renamed from MX487.200; now not fitted
- MX49: renamed from MX364; now not fitted
- MX5: renamed from MX120; now not fitted
- MX51: renamed from MX374; now not fitted
- MX52: renamed from MX375; now not fitted
- MX53: renamed from MX384; now not fitted
- MX54: renamed from MX385; now not fitted
- MX55: renamed from MX407; now not fitted
- MX56: renamed from MX447; now not fitted
- MX57: renamed from MX457; now not fitted
- MX58: renamed from MX467; now not fitted
- MX59: renamed from MX476; now not fitted
- MX6: renamed from MX121; now not fitted
- MX61: renamed from MX477; now not fitted
- MX62: renamed from MX486; now not fitted
- MX63: renamed from MX487; now not fitted
- MX7: renamed from MX130; now not fitted
- MX8: renamed from MX131; now not fitted
- MX9: renamed from MX140; now not fitted
- R1: renamed from R8; LCSC (none) -> C2906948; MPN (none) -> FRC0402J512 TS; Manufacturer (none) -> FOJAN; Original (none) -> N; Purchase Link (none) -> https://www.lcsc.com/product-detail/C2906948.html
- R2: renamed from R9; LCSC (none) -> C2906948; MPN (none) -> FRC0402J512 TS; Manufacturer (none) -> FOJAN; Original (none) -> N; Purchase Link (none) -> https://www.lcsc.com/product-detail/C2906948.html
- R3: renamed from R1; LCSC (none) -> C6460545; MPN (none) -> RT0402FRE07500RL; Manufacturer (none) -> YAGEO; Original (none) -> N; Purchase Link (none) -> https://www.lcsc.com/product-detail/C6460545.html
- R4: renamed from R2; LCSC (none) -> C6460545; MPN (none) -> RT0402FRE07500RL; Manufacturer (none) -> YAGEO; Original (none) -> N; Purchase Link (none) -> https://www.lcsc.com/product-detail/C6460545.html
- RSW2: renamed from RSW181; now not fitted
- S1: renamed from S4; now not fitted
- S2, S5: now not fitted
- S3: renamed from S1; now not fitted
- S4: renamed from S3; now not fitted
- U1: renamed from U5; LCSC (none) -> C81720; MPN (none) -> STM32F072CBT6; Manufacturer (none) -> ST; Original (none) -> Y; Purchase Link (none) -> https://www.lcsc.com/product-detail/C81720.html?s_z=n_STM32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
- U2: MPN (none) -> PRTR5V0U2X; Manufacturer (none) -> TECH PUBLIC; Original (none) -> N; Purchase Link (none) -> https://www.lcsc.com/product-detail/C2827688.html?s_z=n_C28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
- U3: renamed from U4; MPN (none) -> XC6206P332MR-G; Manufacturer (none) -> TOREX; Original (none) -> N; Purchase Link (none) -> https://www.lcsc.com/product-detail/C5446.html?s_z=n_C5446
- U4: renamed from U1; LCSC (none) -> C352970; MPN (none) -> SN74LVC1T45DRLR; Manufacturer (none) -> TI; Original (none) -> N; Purchase Link (none) -> https://www.lcsc.com/product-detail/C352970.html?s_z=n_SN74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
Connections:
- net Col10: now also MX57.1 (COL); no longer MX456.1.1 (COL)
- net Col11: now also MX58.1 (COL); no longer MX57.1 (COL)
- net Col12: now also MX59.1 (COL), MX18.1 (COL); no longer MX58.1 (COL)
- net Col13: now also MX14.1 (COL), MX32.1 (COL), MX50.1 (COL); no longer MX15.1 (COL), MX33.1 (COL), MX51.1 (COL), MX59.1 (COL)
- net Col14: now also MX15.1 (COL), MX33.1 (COL), MX51.1 (COL), MX60.1 (COL); no longer MX16.1 (COL), MX34.1 (COL), MX52.1 (COL), MX61.1 (COL)
- net Col15: now also MX16.1 (COL), MX34.1 (COL), MX52.1 (COL), MX61.1 (COL); no longer MX17.1 (COL), MX35.1 (COL), MX53.1 (COL), MX62.1 (COL)
- net Col16: now also MX17.1 (COL), MX35.1 (COL), MX53.1 (COL), MX62.1 (COL); no longer MX36.1 (COL), MX487.1.1 (COL), MX54.1 (COL), MX63.1 (COL), RSW2.S2
- net Col6: now also MX417.3.1 (COL)
- net Col7: now also MX446.1.1 (COL)
- net Col8: now also MX56.1 (COL); no longer MX446.1.1 (COL)
- net Col9: now also MX456.1.1 (COL); no longer MX56.1 (COL)
- net Row0: now also D36.3 (K)
- net Row1: now also D38.3 (K)
- net Row2: now also D37.3 (K)
- net Row3: now also D34.3 (K)
- net at D7.1 (A), MX13.2 (ROW): now also MX18.2 (ROW)
- net at D30.1 (A), MX417.2.2 (ROW), MX437.1.2 (ROW): now also MX417.3.2 (ROW)
- net at LED34.1 (DO): now also R4.2
- net Col17: now reaches U1.13 (PA3)
- net Col17: now also MX36.1 (COL), MX487.1.1 (COL), MX54.1 (COL), MX63.1 (COL), RSW2.S2
- net Rotary0A: no longer names the net of U1.15 (PA5)
- net Rotary0B: no longer names the net of U1.14 (PA4)
- new net: D34.2 (A), MX61.2 (ROW)
- new net: D34.1 (A), MX477.1.2 (ROW), MX60.2 (ROW)
- new net: D38.2 (A), MX32.2 (ROW)
- new net: D36.2 (A), MX14.2 (ROW)
- new net: D37.2 (A), MX50.2 (ROW)
- now unconnected: D33.2 (A)
- no-connect marks 10 -> 17
Other:
- note added: "5u"
- note added: "LAE"
- moved on the sheet: D17, D18, D26, D27, D31, D32, D33, D35, D8, D9
