File: moin-kastenwagen-plate/moin-kastenwagen-plate.kicad_pcb (KiCad board)
At the start: 2 copper layers, 352.8 x 89 mm, 0 parts

Commit message: Finished Plate v1, Added correct Readme
Parts:
- added Ref**: Val**, silkscreen:GasketHowTo, F.Cu at (561.6, 175.8)
- added Ref**: Val**, silkscreen:GasketHowTo, F.Cu at (250.4, 236.9)
- added Ref**: Val**, silkscreen:GasketHowTo, F.Cu at (246.8, 176.6)
- added Ref**: Val**, silkscreen:Duck 2 with text, F.Cu at (485.9, 175.3)
- added Ref**: Val**, silkscreen:PlanetKastenwagen_10mm, F.Cu at (485.9, 185.1)
- added Ref**: Val**, silkscreen:GasketHowTo, F.Cu at (561.2, 225.8)
- added Ref**: Val**, silkscreen:GasketHowTo, F.Cu at (399.2, 172.6)
- added Ref**: Val**, silkscreen:GasketHowTo, F.Cu at (456.4, 239.3)
Other:
- board size 352.8 x 89 mm -> 351.4 x 87.1 mm
- board text added: "2.25u"
- board text added: "2.75u"
- board text added: "6.25u"
- board text added: "Moin Kastenwagen Alu FR4-Plate v1"

Commit message: PCB und Plate bestellfertig
Parts:
- removed the Ref** at (561.6, 175.8)
- removed the Ref** at (250.4, 236.9)
- removed the Ref** at (246.8, 176.6)
- removed the Ref** at (485.9, 175.3)
- removed the Ref** at (485.9, 185.1)
- removed the Ref** at (561.2, 225.8)
- removed the Ref** at (399.2, 172.6)
Other:
- board size 351.4 x 87.1 mm -> 370.5 x 87.1 mm
- board text added: "1.75 BS"
- board text added: "5u"
- board text added: "LAE"
- board text added: "Moin Kastenwagen Alu BAE Plate v1"
- board text removed: "Moin Kastenwagen Alu FR4-Plate v1"
